Commit message: style: Apply black formatting

File: heron_description/urdf/accessories.urdf.xacro (robot description, xacro)
@@ -34,5 +34,5 @@
     <joint name="$(optenv HERON_NAVSAT_SMART6_MOUNT rear)_navsat_joint" type="fixed">
     <origin xyz="$(optenv HERON_NAVSAT_SMART6_OFFSET -0.25 0 0.08)"
-            rpy="$(optenv HERON_NAVSAT_SMART6_RPY 0 0 0)" />
+        rpy="$(optenv HERON_NAVSAT_SMART6_RPY 0 0 0)" />
       <parent link="$(arg suffix_ns)base_link" />
       <child link="$(arg suffix_ns)$(optenv HERON_NAVSAT_SMART6_MOUNT rear)_navsat" />
@@ -48,5 +48,5 @@
     <joint name="$(optenv HERON_LASER_MOUNT front)_laser_mount_joint" type="fixed">
       <origin xyz="$(optenv HERON_LASER_OFFSET 0.0575 0 0.0115)"
-              rpy="$(optenv HERON_LASER_RPY 0 0 0)" />
+          rpy="$(optenv HERON_LASER_RPY 0 0 0)" />
       <parent link="$(arg suffix_ns)rear_plate" />
       <child link="$(arg suffix_ns)$(optenv HERON_LASER_MOUNT front)_laser_mount" />
@@ -59,5 +59,5 @@
     <joint name="$(optenv HERON_AXIS_PTZ_MOUNT axis_ptz)_camera_joint" type="fixed">
     <origin xyz="$(optenv HERON_AXIS_PTZ_OFFSET -0.124 0 0.078)"
-            rpy="$(optenv HERON_AXIS_PTZ_RPY 0 0 0)" />
+        rpy="$(optenv HERON_AXIS_PTZ_RPY 0 0 0)" />
       <parent link="$(arg suffix_ns)rear_plate" />
       <child link="$(arg suffix_ns)$(optenv HERON_AXIS_PTZ_MOUNT axis_ptz)_camera_link" />
@@ -68,5 +68,5 @@
     <joint name="$(optenv HERON_SONAR_MOUNT rear)_sonar_joint" type="fixed">
     <origin xyz="$(optenv HERON_SONAR_OFFSET 0.0 0 -0.10)"
-            rpy="$(optenv HERON_SONAR_RPY 0 0 0)" />
+        rpy="$(optenv HERON_SONAR_RPY 0 0 0)" />
       <parent link="$(arg suffix_ns)base_link" />
       <child link="$(arg suffix_ns)sonar_$(optenv HERON_SONAR_MOUNT surface)" />

File: heron_description/urdf/base.xacro (robot description, xacro)
@@ -15,72 +15,72 @@
   <material name="yellow"><color rgba="0.8 0.8 0.0 1.0"/></material>
   <xacro:macro name="panel" params="namespace side location">
-      <!-- location flips the panel. 1 is for the left and -1 is for the right -->
-      <joint name="${namespace}base_${side}_joint" type="fixed">
-        <origin xyz="0.0 ${location * 0.34495} 0.04959" rpy="0 0 0" />
-        <parent link="${namespace}base_link" />
-        <child link="${namespace}${side}_panel_link" />
-      </joint>
-      <link name="${namespace}${side}_panel_link">
-        <inertial>
-          <mass value="0.1" />
-          <origin xyz="0.00000000 0.00000000 0.00000000" />
-          <inertia ixx="0.01" ixy="0.00" ixz="0.00"
-            iyy="0.01" iyz="0.00" izz="0.01" />
-        </inertial>
-        <visual>
-          <origin xyz="0 0 0" rpy="0 0 0" />
-          <geometry>
-            <mesh filename="package://heron_description/meshes/${side}_panel.stl" />
-          </geometry>
-          <material name="yellow" />
-        </visual>
-      </link>
-      <gazebo reference="${namespace}${side}_panel_link">
-        <material>Gazebo/Yellow</material>
-      </gazebo>
+    <!-- location flips the panel. 1 is for the left and -1 is for the right -->
+    <joint name="${namespace}base_${side}_joint" type="fixed">
+      <origin xyz="0.0 ${location * 0.34495} 0.04959" rpy="0 0 0" />
+      <parent link="${namespace}base_link" />
+      <child link="${namespace}${side}_panel_link" />
+    </joint>
+    <link name="${namespace}${side}_panel_link">
+      <inertial>
+        <mass value="0.1" />
+        <origin xyz="0.00000000 0.00000000 0.00000000" />
+        <inertia ixx="0.01" ixy="0.00" ixz="0.00"
+          iyy="0.01" iyz="0.00" izz="0.01" />
+      </inertial>
+      <visual>
+        <origin xyz="0 0 0" rpy="0 0 0" />
+        <geometry>
+          <mesh filename="package://heron_description/meshes/${side}_panel.stl" />
+        </geometry>
+        <material name="yellow" />
+      </visual>
+    </link>
+    <gazebo reference="${namespace}${side}_panel_link">
+      <material>Gazebo/Yellow</material>
+    </gazebo>
     </xacro:macro>
   <!-- Vehicle macro -->
   <xacro:macro name="heron_base" params="namespace *gazebo">
-      <link name="${namespace}base_footprint"/>
-      <joint name="${namespace}base_footprint_joint" type="fixed">
-        <origin xyz="0 0 0" rpy="0 0 0" />
-        <parent link="${namespace}base_footprint" />
-        <child link="${namespace}base_link" />
-      </joint>
-      <!-- Rigid body description of the base link -->
-      <link name="${namespace}base_link">
-        <!--
-          Be careful to setup the coefficients for the inertial tensor,
-          otherwise your model will become unstable on Gazebo
-        -->
-        <visual>
-          <origin xyz="0 0 0" rpy="0 0 0"/>
-          <geometry>
-            <mesh filename="package://heron_description/meshes/heron_base.stl" scale="1 1 1" />
-          </geometry>
-          <material name="dark_gray" />
-        </visual>
-        <collision>
-          <origin xyz="0 0 0" rpy="0 0 0"/>
-          <geometry>
-            <mesh filename="package://heron_description/meshes/heron_collision.stl" scale="1 1 1" />
-          </geometry>
-        </collision>
-      </link>
-      <!-- Dummy Link to contain the inertial information for base_link -->
-      <link name="${namespace}dummy_link">
-        <inertial>
-          <mass value="${mass}" />
-          <origin xyz="${cog}" rpy="0 0 0"/>
-          <inertia ixx="10" ixy="0" iyy = "10" ixz="0" iyz="0" izz="10" />
-          <!-- <inertia ixx="0.017474" ixy="-0.000013" ixz="-0.000102"
-                                  iyy="0.017781"  iyz="-0.000058"
-                                                  izz="0.033235" /> -->
-        </inertial>
-      </link>
-      <joint name="dummy_to_base" type="fixed">
-        <parent link="${namespace}base_link" />
-        <child link="${namespace}dummy_link" />
-      </joint>
+    <link name="${namespace}base_footprint"/>
+    <joint name="${namespace}base_footprint_joint" type="fixed">
+      <origin xyz="0 0 0" rpy="0 0 0" />
+      <parent link="${namespace}base_footprint" />
+      <child link="${namespace}base_link" />
+    </joint>
+    <!-- Rigid body description of the base link -->
+    <link name="${namespace}base_link">
+      <!--
+        Be careful to setup the coefficients for the inertial tensor,
+        otherwise your model will become unstable on Gazebo
+      -->
+      <visual>
+        <origin xyz="0 0 0" rpy="0 0 0"/>
+        <geometry>
+          <mesh filename="package://heron_description/meshes/heron_base.stl" scale="1 1 1" />
+        </geometry>
+        <material name="dark_gray" />
+      </visual>
+      <collision>
+        <origin xyz="0 0 0" rpy="0 0 0"/>
+        <geometry>
+          <mesh filename="package://heron_description/meshes/heron_collision.stl" scale="1 1 1" />
+        </geometry>
+      </collision>
+    </link>
+    <!-- Dummy Link to contain the inertial information for base_link -->
+    <link name="${namespace}dummy_link">
+      <inertial>
+        <mass value="${mass}" />
+        <origin xyz="${cog}" rpy="0 0 0"/>
+        <inertia ixx="10" ixy="0" iyy = "10" ixz="0" iyz="0" izz="10" />
+        <!-- <inertia ixx="0.017474" ixy="-0.000013" ixz="-0.000102"
+                    iyy="0.017781"  iyz="-0.000058"
+                            izz="0.033235" /> -->
+      </inertial>
+    </link>
+    <joint name="dummy_to_base" type="fixed">
+      <parent link="${namespace}base_link" />
+      <child link="${namespace}dummy_link" />
+    </joint>
     <gazebo reference="${namespace}base_link">
       <selfCollide>false</selfCollide>

File: heron_description/urdf/gazebo.xacro (robot description, xacro)
@@ -1,62 +1,62 @@
 <?xml version="1.0"?>
 <robot xmlns:xacro="http://www.ros.org/wiki/xacro">
-    <!-- Center of buoyancy -->
-    <xacro:property name="heron_cob" value="0 0 0"/>
-    <!-- Vehicle's actual volume (Gazebo cannot compute the volume out of the mesh) -->
-    <xacro:property name="heron_volume" value="0.13"/>
-    <!-- Describing the dimensions of the vehicle's bounding box -->
-    <xacro:property name="heron_length" value="1.35"/>
-    <xacro:property name="heron_width"  value="1.0"/>
-    <xacro:property name="heron_height" value="0.32"/>
-    <xacro:macro name="heron_hydro_model" params="namespace">
-      <!-- List of hydrodynamic models this robot's links -->
-      <link name="${namespace}base_link">
-              <volume>${heron_volume}</volume>
-              <box>
-                  <width>${heron_width}</width>
-                  <length>${heron_length}</length>
-                  <height>${heron_height}</height>
-              </box>
-              <center_of_buoyancy>${heron_cob}</center_of_buoyancy>
-              <!-- Parameters used to describe the buoyancy force computation
-                   for the surface vessel as implemented in the custom force
-                   translation plugin.
-              -->
-              <metacentric_width>0.1</metacentric_width>
-              <metacentric_length>0.1</metacentric_length>
-              <submerged_height>0.02</submerged_height>
-              <hydrodynamic_model>
-                  <type>fossen</type>
-                  <added_mass>
-                     0   0   0   0   0   0
-                     0   0   0   0   0   0
-                     0   0   0   0   0   0
-                     0   0   0   0   0   0
-                     0   0   0   0   0   0
-                     0   0   0   0   0   0
-                </added_mass>
-                <offset_added_mass>0</offset_added_mass>
-                <linear_damping>
-                      -25 -24 -150 -20 -20 -10
-                  </linear_damping>
-                  <quadratic_damping>
-                    -5 -5 -15 -8 -8 -8
-                  </quadratic_damping>
-                  <!-- Sanity check -->
-                  <linear_damping_forward_speed>
-                    0 0 0 0 0 0
-                  </linear_damping_forward_speed>
-                  <offset_linear_damping>
-                    0
-                  </offset_linear_damping>
-                  <offset_lin_forward_speed_damping>
-                    0
-                  </offset_lin_forward_speed_damping>
-                  <offset_nonlin_damping>
-                    0
-                  </offset_nonlin_damping>
-                  <scaling_damping>1.0</scaling_damping>
-              </hydrodynamic_model>
-          </link>
-    </xacro:macro>
+  <!-- Center of buoyancy -->
+  <xacro:property name="heron_cob" value="0 0 0"/>
+  <!-- Vehicle's actual volume (Gazebo cannot compute the volume out of the mesh) -->
+  <xacro:property name="heron_volume" value="0.13"/>
+  <!-- Describing the dimensions of the vehicle's bounding box -->
+  <xacro:property name="heron_length" value="1.35"/>
+  <xacro:property name="heron_width"  value="1.0"/>
+  <xacro:property name="heron_height" value="0.32"/>
+  <xacro:macro name="heron_hydro_model" params="namespace">
+    <!-- List of hydrodynamic models this robot's links -->
+    <link name="${namespace}base_link">
+        <volume>${heron_volume}</volume>
+        <box>
+          <width>${heron_width}</width>
+          <length>${heron_length}</length>
+          <height>${heron_height}</height>
+        </box>
+        <center_of_buoyancy>${heron_cob}</center_of_buoyancy>
+        <!-- Parameters used to describe the buoyancy force computation
+             for the surface vessel as implemented in the custom force
+             translation plugin.
+        -->
+        <metacentric_width>0.1</metacentric_width>
+        <metacentric_length>0.1</metacentric_length>
+        <submerged_height>0.02</submerged_height>
+        <hydrodynamic_model>
+          <type>fossen</type>
+          <added_mass>
+             0   0   0   0   0   0
+             0   0   0   0   0   0
+             0   0   0   0   0   0
+             0   0   0   0   0   0
+             0   0   0   0   0   0
+             0   0   0   0   0   0
+          </added_mass>
+          <offset_added_mass>0</offset_added_mass>
+          <linear_damping>
+                -25 -24 -150 -20 -20 -10
+            </linear_damping>
+            <quadratic_damping>
+              -5 -5 -15 -8 -8 -8
+            </quadratic_damping>
+            <!-- Sanity check -->
+            <linear_damping_forward_speed>
+              0 0 0 0 0 0
+            </linear_damping_forward_speed>
+            <offset_linear_damping>
+              0
+            </offset_linear_damping>
+            <offset_lin_forward_speed_damping>
+              0
+            </offset_lin_forward_speed_damping>
+            <offset_nonlin_damping>
+              0
+            </offset_nonlin_damping>
+            <scaling_damping>1.0</scaling_damping>
+        </hydrodynamic_model>
+      </link>
+  </xacro:macro>
 </robot>

File: heron_description/urdf/heron.urdf.xacro (robot description, xacro)
@@ -5,12 +5,12 @@
 Redistribution and use in source and binary forms, with or without
 modification, are permitted provided that the following conditions are met:
-    * Redistributions of source code must retain the above copyright
-      notice, this list of conditions and the following disclaimer.
-    * Redistributions in binary form must reproduce the above copyright
-      notice, this list of conditions and the following disclaimer in the
-      documentation and/or other materials provided with the distribution.
-    * Neither the name of Clearpath Robotics nor the
-      names of its contributors may be used to endorse or promote products
-      derived from this software without specific prior written permission.
+  * Redistributions of source code must retain the above copyright
+    notice, this list of conditions and the following disclaimer.
+  * Redistributions in binary form must reproduce the above copyright
+    notice, this list of conditions and the following disclaimer in the
+    documentation and/or other materials provided with the distribution.
+  * Neither the name of Clearpath Robotics nor the
+    names of its contributors may be used to endorse or promote products
+    derived from this software without specific prior written permission.
 THIS SOFTWARE IS PROVIDED BY THE COPYRIGHT HOLDERS AND CONTRIBUTORS "AS IS" AND
 ANY EXPRESS OR IMPLIED WARRANTIES, INCLUDING, BUT NOT LIMITED TO, THE IMPLIED
