Commit message: Continue Heron ROS 2 port

File: heron_description/urdf/accessories.urdf.xacro (robot description, xacro)
@@ -24,7 +24,4 @@
       <origin xyz="-0.1915 0.0 0.001" />
     </joint>
-    <gazebo reference="${suffix_ns}rear_plate">
-      <material>Gazebo/DarkGrey</material>
-    </gazebo>
   </xacro:macro>
   <!-- If enabled, generate a Novatel Smart6 payload. -->

File: heron_description/urdf/accessories/sick_lms1xx_mount.urdf.xacro (robot description, xacro)
@@ -11,7 +11,4 @@
       <child link="${suffix_ns}${prefix}_laser" />
     </joint>
-    <gazebo reference="${suffix_ns}${prefix}_laser_mount">
-      <material>Gazebo/DarkGrey</material>
-    </gazebo>
   </xacro:macro>
 </robot>

File: heron_description/urdf/base.xacro (robot description, xacro)
@@ -39,7 +39,4 @@
       </visual>
     </link>
-    <gazebo reference="${namespace}${side}_panel_link">
-      <material>Gazebo/Yellow</material>
-    </gazebo>
     </xacro:macro>
   <!-- Vehicle macro -->
@@ -88,5 +85,4 @@
     <gazebo reference="${namespace}base_link">
       <selfCollide>false</selfCollide>
-      <material>Gazebo/DarkGrey</material>
       <gravity>1</gravity>
     </gazebo>
@@ -94,10 +90,10 @@
     <xacro:insert_block name="gazebo"/>
     <!-- Include the thruster modules -->
-    <xacro:thruster_macro robot_namespace="$(arg namespace)" suffix_ns="$(arg suffix_ns)" thruster_id="0"
+    <xacro:thruster_macro robot_namespace="$(arg namespace)" suffix_ns="$(arg suffix_ns)" thruster_id="0" side="right"
       simulation="$(arg simulation)">
       <!-- Right Thruster -->
       <origin xyz="-0.53 -0.377654 -0.16" rpy="0 0 0" />
     </xacro:thruster_macro>
-    <xacro:thruster_macro robot_namespace="$(arg namespace)" suffix_ns="$(arg suffix_ns)" thruster_id="1"
+    <xacro:thruster_macro robot_namespace="$(arg namespace)" suffix_ns="$(arg suffix_ns)" thruster_id="1" side="left"
       simulation="$(arg simulation)">
       <!-- Left Thruster -->
@@ -108,5 +104,5 @@
     <xacro:panel namespace="$(arg suffix_ns)" side="left" location="1" />
     <xacro:panel namespace="$(arg suffix_ns)" side="right" location="-1" />
-    <xacro:include filename="$(find heron_description)/urdf/accessories.urdf.xacro" />
+  <xacro:include filename="$(find heron_description)/urdf/accessories.urdf.xacro" />
     <!-- Optional custom includes. -->
     <xacro:include filename="$(optenv HERON_URDF_EXTRAS empty.urdf)" />

File: heron_description/urdf/heron.urdf.xacro (robot description, xacro)
@@ -58,8 +58,8 @@
   <!-- Create the heron -->
   <xacro:heron_base namespace="$(arg suffix_ns)">
-    <!-- Keep the surface vessel at its waterline with an owned Noetic/Gazebo
+    <!-- Keep the surface vessel at its waterline with an owned Gazebo Sim
          model. This replaces the obsolete external UUV Simulator plugin. -->
     <gazebo>
-      <plugin name="surface_hydrodynamics" filename="libSurfaceHydrodynamicsPlugin.so">
+      <plugin name="grande::simulation::SurfaceHydrodynamicsPlugin" filename="libSurfaceHydrodynamicsPlugin.so">
         <bodyName>$(arg suffix_ns)base_footprint</bodyName>
         <equilibriumZ>0.0</equilibriumZ>
@@ -79,5 +79,5 @@
        boat. Canonical integrated bringup does not publish this topic. -->
   <gazebo>
-    <plugin name="hydrodynamic_forces" filename="libRelativeForcePlugin.so">
+    <plugin name="grande::simulation::RelativeForcePlugin" filename="libRelativeForcePlugin.so">
       <bodyName>$(arg suffix_ns)base_link</bodyName>
       <commandTimeout>0.5</commandTimeout>
@@ -91,5 +91,5 @@
   </gazebo>
   <gazebo>
-    <plugin name="passive_disturbance" filename="libPassiveDisturbancePlugin.so">
+    <plugin name="grande::simulation::PassiveDisturbancePlugin" filename="libPassiveDisturbancePlugin.so">
       <bodyName>$(arg suffix_ns)base_link</bodyName>
       <forceMean>${disturbance_force_mean_x} ${disturbance_force_mean_y} ${disturbance_force_mean_z}</forceMean>
@@ -100,15 +100,25 @@
     </plugin>
   </gazebo>
-  <!-- Joint state publisher plugin -->
+  <!-- Gazebo Sim publishes joint state in Gazebo Transport. ros_gz_bridge
+       exposes it as /joint_states for robot_state_publisher. -->
   <gazebo>
-    <plugin name="joint_state_publisher" filename="libgazebo_ros_joint_state_publisher.so">
-      <xacro:if value="${'$(arg namespace)' != ''}">
-        <robotNamespace>/$(arg namespace)</robotNamespace>
-      </xacro:if>
-      <xacro:unless value="${'$(arg namespace)' != ''}">
-        <robotNamespace></robotNamespace>
-      </xacro:unless>
-      <updateRate>10</updateRate>
-      <jointName>thruster_0_joint, thruster_1_joint</jointName>
+    <plugin name="gz::sim::systems::JointStatePublisher"
+            filename="gz-sim-joint-state-publisher-system">
+      <topic>/joint_states</topic>
+      <joint_name>$(arg suffix_ns)thruster_0_joint</joint_name>
+      <joint_name>$(arg suffix_ns)thruster_1_joint</joint_name>
+    </plugin>
+  </gazebo>
+  <!-- Ground truth is exposed for labelled simulation/evaluation only. It is
+       not an estimator or navigation feedback source. -->
+  <gazebo>
+    <plugin name="gz::sim::systems::OdometryPublisher"
+            filename="gz-sim-odometry-publisher-system">
+      <odom_frame>world</odom_frame>
+      <robot_base_frame>$(arg suffix_ns)base_link</robot_base_frame>
+      <odom_publish_frequency>20</odom_publish_frequency>
+      <odom_topic>/pose_gt</odom_topic>
+      <dimensions>3</dimensions>
+      <gaussian_noise>0.0</gaussian_noise>
     </plugin>
   </gazebo>

File: heron_description/urdf/sensors.xacro (robot description, xacro)
@@ -2,20 +2,26 @@
 <robot xmlns:xacro="http://www.ros.org/wiki/xacro">
   <!-- GPS -->
-  <gazebo>
-    <plugin name="gps_controller" filename="libhector_gazebo_ros_gps.so">
-      <updateRate>40</updateRate>
-      <robotNamespace>/$(arg namespace)</robotNamespace>
-      <frameId>$(arg suffix_ns)navsat_link</frameId>
-      <bodyName>$(arg suffix_ns)navsat_link</bodyName>
-      <topicName>/$(arg suffix_ns)navsat/fix</topicName>
-      <velocityTopicName>/$(arg suffix_ns)navsat/velocity</velocityTopicName>
-      <referenceLatitude>49.9</referenceLatitude>
-      <referenceLongitude>8.9</referenceLongitude>
-      <referenceHeading>90</referenceHeading>
-      <referenceAltitude>0</referenceAltitude>
-      <drift>0.0001 0.0001 0.0001</drift>
-    </plugin>
+  <link name="$(arg suffix_ns)navsat_link" />
+  <gazebo reference="$(arg suffix_ns)navsat_link">
+    <sensor name="heron_navsat" type="navsat">
+      <always_on>true</always_on>
+      <update_rate>40</update_rate>
+      <topic>/navsat/fix</topic>
+      <navsat>
+        <position_sensing>
+          <horizontal>
+            <noise type="gaussian">
+              <stddev>0.0001</stddev>
+            </noise>
+          </horizontal>
+          <vertical>
+            <noise type="gaussian">
+              <stddev>0.0001</stddev>
+            </noise>
+          </vertical>
+        </position_sensing>
+      </navsat>
+    </sensor>
   </gazebo>
-  <link name="$(arg suffix_ns)navsat_link" />
   <joint name="navsat_joint" type="fixed">
     <parent link="$(arg suffix_ns)base_link" />
@@ -25,20 +31,24 @@
     </joint>
     <!-- IMU -->
-    <gazebo>
-      <plugin name="imu_controller" filename="libhector_gazebo_ros_imu.so">
-        <robotNamespace>/$(arg namespace)</robotNamespace>
-        <updateRate>50.0</updateRate>
-        <bodyName>$(arg suffix_ns)imu_link</bodyName>
-        <frameId>$(arg suffix_ns)imu_link</frameId>
-        <topicName>/$(arg suffix_ns)imu/data_raw</topicName>
-        <accelDrift>0.005 0.005 0.005</accelDrift>
-        <accelGaussianNoise>0.005 0.005 0.005</accelGaussianNoise>
-        <rateDrift>0.005 0.005 0.005 </rateDrift>
-        <rateGaussianNoise>0.005 0.005 0.005 </rateGaussianNoise>
-        <headingDrift>0.005</headingDrift>
-        <headingGaussianNoise>0.005</headingGaussianNoise>
-      </plugin>
+    <link name="$(arg suffix_ns)imu_link" />
+    <gazebo reference="$(arg suffix_ns)imu_link">
+      <sensor name="heron_raw_imu" type="imu">
+        <always_on>true</always_on>
+        <update_rate>50</update_rate>
+        <topic>/imu/data_raw</topic>
+        <imu>
+          <angular_velocity>
+            <x><noise type="gaussian"><stddev>0.005</stddev></noise></x>
+            <y><noise type="gaussian"><stddev>0.005</stddev></noise></y>
+            <z><noise type="gaussian"><stddev>0.005</stddev></noise></z>
+          </angular_velocity>
+          <linear_acceleration>
+            <x><noise type="gaussian"><stddev>0.005</stddev></noise></x>
+            <y><noise type="gaussian"><stddev>0.005</stddev></noise></y>
+            <z><noise type="gaussian"><stddev>0.005</stddev></noise></z>
+          </linear_acceleration>
+        </imu>
+      </sensor>
     </gazebo>
-    <link name="$(arg suffix_ns)imu_link" />
     <joint name="$(arg suffix_ns)imu_joint" type="fixed">
       <origin xyz="$(optenv HERON_IMU_XYZ -0.1397 0.0 0)" rpy="$(optenv HERON_IMU_RPY 0 0.0 0.0)" />
@@ -47,29 +57,15 @@
     </joint>
     <!-- Magnetometer -->
-    <gazebo>
-      <plugin name="mag_controller" filename="libhector_gazebo_ros_magnetic.so">
-        <updateRate>50</updateRate>
-        <robotNamespace>/$(arg namespace)</robotNamespace>
-        <bodyName>$(arg suffix_ns)imu_link</bodyName>
-        <frameId>$(arg suffix_ns)imu_link</frameId>
-        <topicName>/$(arg suffix_ns)imu/mag_raw</topicName>
-        <referenceHeading>90</referenceHeading>
-        <drift>0.0005 0.0005 0.0005</drift>
-        <gaussianNoise>0.025 0.025 0.025</gaussianNoise>
-        <useMagneticFieldMsgs>false</useMagneticFieldMsgs>
-      </plugin>
-    </gazebo>
-    <!-- Mount a Perfect Pose 3D sensor. -->
-    <gazebo>
-      <plugin filename="libgazebo_ros_p3d.so" name="groundtruth_sim">
-        <updateRate>20.0</updateRate>
-        <robotNamespace>/$(arg namespace)</robotNamespace>
-        <bodyName>$(arg suffix_ns)base_link</bodyName>
-        <topicName>/$(arg suffix_ns)pose_gt</topicName>
-        <gaussianNoise>0.0</gaussianNoise>
-        <!-- Gazebo publishes a world pose; label it truthfully and transform it
-             only in evaluation using the declared scenario spawn pose. -->
-        <frameName>world</frameName>
-      </plugin>
+    <gazebo reference="$(arg suffix_ns)imu_link">
+      <sensor name="heron_magnetometer" type="magnetometer">
+        <always_on>true</always_on>
+        <update_rate>50</update_rate>
+        <topic>/imu/mag_raw</topic>
+        <magnetometer>
+          <x><noise type="gaussian"><stddev>0.025</stddev></noise></x>
+          <y><noise type="gaussian"><stddev>0.025</stddev></noise></y>
+          <z><noise type="gaussian"><stddev>0.025</stddev></noise></z>
+        </magnetometer>
+      </sensor>
     </gazebo>
   </robot>

File: heron_description/urdf/snippets.xacro (robot description, xacro)
@@ -6,5 +6,5 @@
     be initialized in the actuators.xacro file.
   -->
-  <xacro:macro name="thruster_macro" params="robot_namespace suffix_ns thruster_id *origin simulation:=false">
+  <xacro:macro name="thruster_macro" params="robot_namespace suffix_ns thruster_id side *origin simulation:=false">
     <!--
     Dummy link as place holder for the thruster frame,
@@ -35,15 +35,13 @@
       </joint>
       <gazebo>
-        <!-- Apply thrust in the thruster link frame. The stock gazebo_ros_force
-             plugin applies world-frame force, which makes the hull yaw while
-             still being pushed in a stale global direction. -->
-        <plugin name="${robot_namespace}thruster_${thruster_id}_model" filename="libRelativeForcePlugin.so">
+        <!-- The Gazebo Sim system applies thrust in the thruster link frame. -->
+        <plugin name="grande::simulation::RelativeForcePlugin" filename="libRelativeForcePlugin.so">
           <bodyName>${suffix_ns}thruster_${thruster_id}</bodyName>
           <commandTimeout>0.5</commandTimeout>
           <xacro:if value="${robot_namespace != ''}">
-            <topicName>/${robot_namespace}/thrusters/${thruster_id}/input</topicName>
+            <topicName>/${robot_namespace}/thrusters/${side}/input</topicName>
           </xacro:if>
           <xacro:unless value="${robot_namespace != ''}">
-            <topicName>/thrusters/${thruster_id}/input</topicName>
+            <topicName>/thrusters/${side}/input</topicName>
           </xacro:unless>
         </plugin>
