Commit message: Refactor: Remove UUV dependencies and update for Noetic
- Updated CHANGELOGs.
- Updated heron_control launch files and scripts.
- Purged UUV references in heron_description.

File: heron_description/urdf/gazebo.xacro (robot description, xacro)
@@ -19,7 +19,7 @@
               </box>
               <center_of_buoyancy>${heron_cob}</center_of_buoyancy>
-              <!-- The buoyancy plugin in the UUV Simulator can then be adapted
-                   to receive the additional parameters used to describe the
-                   buoyancy force computation for the surface vessel.
+              <!-- Parameters used to describe the buoyancy force computation
+                   for the surface vessel as implemented in the custom force
+                   translation plugin.
               -->
               <metacentric_width>0.1</metacentric_width>

File: heron_description/urdf/heron.urdf.xacro (robot description, xacro)
@@ -37,25 +37,19 @@
      allow the addition of external models of manipulator units -->
     <gazebo>
-      <plugin name="uuv_plugin" filename="libuuv_underwater_object_ros_plugin.so">
-        <fluid_density>1028.0</fluid_density>
-        <flow_velocity_topic>hydrodynamics/current_velocity</flow_velocity_topic>
-        <debug>$(arg debug)</debug>
-        <!-- Adding the hydrodynamic and hydrostatic parameters for the vehicle-->
-        <xacro:heron_hydro_model namespace="$(arg suffix_ns)" />
-        <!--
-          In case other modules are added to the vehicle (such as a manipulator)
-          that also have link running with the underwater object plugin, they
-          should also be added in this block. For this, this new module should
-          have a file similar to gazebo.xacro above with the description of the
-          parameter necessary for the underwater object plugin to be initialized.
-        -->
-      </plugin>
     </gazebo>
   </xacro:heron_base>
+  <!-- Hydrodynamic force plugin (to be driven by vessel_dynamics node) -->
+  <gazebo>
+    <plugin name="hydrodynamic_forces" filename="libgazebo_ros_force.so">
+      <bodyName>$(arg suffix_ns)base_link</bodyName>
+      <topicName>/$(arg namespace)/hydro_forces</topicName>
+    </plugin>
+  </gazebo>
   <!-- Joint state publisher plugin -->
   <gazebo>
-    <plugin name="joint_state_publisher" filename="libuuv_joint_state_publisher.so">
+    <plugin name="joint_state_publisher" filename="libgazebo_ros_joint_state_publisher.so">
       <robotNamespace>/$(arg namespace)</robotNamespace>
       <updateRate>10</updateRate>
+      <jointName>thruster_0_joint, thruster_1_joint</jointName>
     </plugin>
   </gazebo>

File: heron_description/urdf/snippets.xacro (robot description, xacro)
@@ -35,49 +35,8 @@
       </joint>
       <gazebo>
-        <!-- Thruster ROS plugin -->
-        <plugin name="${robot_namespace}thruster_${thruster_id}_thruster_model" filename="libuuv_thruster_ros_plugin.so">
-          <!-- Name of the thruster link -->
-          <linkName>${suffix_ns}thruster_${thruster_id}</linkName>
-          <!-- Name of the joint between thruster and vehicle base link -->
-          <jointName>${suffix_ns}thruster_${thruster_id}_joint</jointName>
-          <!-- Make the thruster aware of its id -->
-          <thrusterID>${thruster_id}</thrusterID>
-          <!-- Gain of the input command signal -->
-          <gain>1</gain>
-          <!-- Maximum allowed input value for the input signal for thruster unit -->
-          <clampMax>100</clampMax>
-          <!-- Minimum allowed value for the input signal for thruster unit -->
-          <clampMin>-100</clampMin>
-          <!-- Minimum and maximum thrust force output allowed -->
-          <thrustMin>-35</thrustMin>
-          <thrustMax>35</thrustMax>
-          <!--
-          Value from 0 to 1 to set the efficiency of the output thrust force
-          Default value is 1.0
-          -->
-          <thrust_efficiency>1</thrust_efficiency>
-          <!--
-          Value from 0 to 1 to set the efficiency of the propeller as a factor
-          to be multiplied to the current value of the state variable at each
-          iteration.
-          Default value is 1.0
-          -->
-          <propeller_efficiency>1</propeller_efficiency>
-          <!-- 2) First order model -->
-          <dynamics>
-            <type>FirstOrder</type>
-            <timeConstant>0.05</timeConstant>
-          </dynamics>
-          <!-- 3) Linear interpolation
-          If you have access to the thruster's data sheet, for example,
-          you can enter samples of the curve's input and output values
-          and the thruster output will be found through linear interpolation
-          of the given samples.
-          -->
-          <conversion>
-            <type>LinearInterp</type>
-            <inputValues>-1.0 -0.8 -0.6 -0.4 -0.2 0 0.2 0.4 0.6 0.8 1.0</inputValues>
-            <outputValues>-19.88 -16.52 -12.6 -5.6 -1.4 0.0 2.24 9.52 21.28 28.0 33.6</outputValues>
-          </conversion>
+        <!-- Thruster force plugin using standard Gazebo -->
+        <plugin name="${robot_namespace}thruster_${thruster_id}_model" filename="libgazebo_ros_force.so">
+          <bodyName>${suffix_ns}thruster_${thruster_id}</bodyName>
+          <topicName>/${robot_namespace}/thrusters/${thruster_id}/input</topicName>
         </plugin>
       </gazebo>

Commit message: feat: Integrate UUV Gazebo plugins, refine namespace handling for thrusters, add startup delays to control nodes, and conditionally launch interactive markers.

File: heron_description/urdf/gazebo.xacro (robot description, xacro)
@@ -11,5 +11,8 @@
   <xacro:macro name="heron_hydro_model" params="namespace">
     <!-- List of hydrodynamic models this robot's links -->
-    <link name="${namespace}base_link">
+      <!-- Gazebo collapses the fixed-joint hull chain into base_footprint when
+           converting this URDF to SDF, so hydrodynamic plugins must target the
+           physical link name instead of the TF frame name base_link. -->
+      <link name="${namespace}base_footprint">
         <volume>${heron_volume}</volume>
         <box>

File: heron_description/urdf/heron.urdf.xacro (robot description, xacro)
@@ -37,4 +37,9 @@
      allow the addition of external models of manipulator units -->
     <gazebo>
+      <plugin name="uuv_plugin" filename="libuuv_underwater_object_ros_plugin.so">
+        <fluid_density>997.7735</fluid_density>
+        <debug>$(arg debug)</debug>
+        <xacro:heron_hydro_model namespace="$(arg suffix_ns)"/>
+      </plugin>
     </gazebo>
   </xacro:heron_base>
@@ -58,5 +63,5 @@
       </xacro:if>
       <xacro:unless value="${'$(arg namespace)' != ''}">
-        <robotNamespace>/</robotNamespace>
+        <robotNamespace></robotNamespace>
       </xacro:unless>
       <updateRate>10</updateRate>

File: heron_description/urdf/snippets.xacro (robot description, xacro)
@@ -38,5 +38,10 @@
         <plugin name="${robot_namespace}thruster_${thruster_id}_model" filename="libgazebo_ros_force.so">
           <bodyName>${suffix_ns}thruster_${thruster_id}</bodyName>
-          <topicName>/${robot_namespace}/thrusters/${thruster_id}/input</topicName>
+          <xacro:if value="${robot_namespace != ''}">
+            <topicName>/${robot_namespace}/thrusters/${thruster_id}/input</topicName>
+          </xacro:if>
+          <xacro:unless value="${robot_namespace != ''}">
+            <topicName>/thrusters/${thruster_id}/input</topicName>
+          </xacro:unless>
         </plugin>
       </gazebo>
