Commit message: chore: sync changes

File: heron_description/urdf/base.xacro (robot description, xacro)
@@ -42,4 +42,10 @@
   <!-- Vehicle macro -->
   <xacro:macro name="heron_base" params="namespace *gazebo">
+      <link name="${namespace}base_footprint"/>
+      <joint name="${namespace}base_footprint_joint" type="fixed">
+        <origin xyz="0 0 0" rpy="0 0 0" />
+        <parent link="${namespace}base_footprint" />
+        <child link="${namespace}base_link" />
+      </joint>
       <!-- Rigid body description of the base link -->
       <link name="${namespace}base_link">

Commit message: feat: tune ig-handle benchmark hull

File: heron_description/urdf/base.xacro (robot description, xacro)
@@ -4,5 +4,8 @@
     Vehicle's parameters (remember to enter the model parameters below)
   -->
-  <xacro:property name="mass" value="28"/>
+  <xacro:property name="base_mass" value="$(optenv HERON_BASE_MASS 28.0)"/>
+  <xacro:property name="base_inertia_ixx" value="$(optenv HERON_BASE_INERTIA_IXX 10.0)"/>
+  <xacro:property name="base_inertia_iyy" value="$(optenv HERON_BASE_INERTIA_IYY 10.0)"/>
+  <xacro:property name="base_inertia_izz" value="$(optenv HERON_BASE_INERTIA_IZZ 10.0)"/>
   <!-- Center of gravity -->
   <xacro:property name="cog" value="0 0 -0.13"/>
@@ -71,7 +74,7 @@
     <link name="${namespace}dummy_link">
       <inertial>
-        <mass value="${mass}" />
+        <mass value="${base_mass}" />
         <origin xyz="${cog}" rpy="0 0 0"/>
-        <inertia ixx="10" ixy="0" iyy = "10" ixz="0" iyz="0" izz="10" />
+        <inertia ixx="${base_inertia_ixx}" ixy="0" iyy="${base_inertia_iyy}" ixz="0" iyz="0" izz="${base_inertia_izz}" />
         <!-- <inertia ixx="0.017474" ixy="-0.000013" ixz="-0.000102"
                     iyy="0.017781"  iyz="-0.000058"
@@ -100,5 +103,5 @@
       <!-- Left Thruster -->
       <origin xyz="-0.53 0.377654 -0.16" rpy="0 0 0" />
-    </xacro:thruster_macro>s
+    </xacro:thruster_macro>
     <!-- Include the sensor modules -->
     <xacro:include filename="$(find heron_description)/urdf/sensors.xacro"/>

File: heron_description/urdf/gazebo.xacro (robot description, xacro)
@@ -9,4 +9,22 @@
   <xacro:property name="heron_width"  value="1.0"/>
   <xacro:property name="heron_height" value="0.32"/>
+  <xacro:property name="added_mass_x" value="$(optenv HERON_ADDED_MASS_X 0.0)"/>
+  <xacro:property name="added_mass_y" value="$(optenv HERON_ADDED_MASS_Y 0.0)"/>
+  <xacro:property name="added_mass_z" value="$(optenv HERON_ADDED_MASS_Z 0.0)"/>
+  <xacro:property name="added_mass_roll" value="$(optenv HERON_ADDED_MASS_ROLL 0.0)"/>
+  <xacro:property name="added_mass_pitch" value="$(optenv HERON_ADDED_MASS_PITCH 0.0)"/>
+  <xacro:property name="added_mass_yaw" value="$(optenv HERON_ADDED_MASS_YAW 0.0)"/>
+  <xacro:property name="linear_damping_x" value="$(optenv HERON_LINEAR_DAMPING_X -25.0)"/>
+  <xacro:property name="linear_damping_y" value="$(optenv HERON_LINEAR_DAMPING_Y -24.0)"/>
+  <xacro:property name="linear_damping_z" value="$(optenv HERON_LINEAR_DAMPING_Z -150.0)"/>
+  <xacro:property name="linear_damping_roll" value="$(optenv HERON_LINEAR_DAMPING_ROLL -20.0)"/>
+  <xacro:property name="linear_damping_pitch" value="$(optenv HERON_LINEAR_DAMPING_PITCH -20.0)"/>
+  <xacro:property name="linear_damping_yaw" value="$(optenv HERON_LINEAR_DAMPING_YAW -10.0)"/>
+  <xacro:property name="quadratic_damping_x" value="$(optenv HERON_QUADRATIC_DAMPING_X -5.0)"/>
+  <xacro:property name="quadratic_damping_y" value="$(optenv HERON_QUADRATIC_DAMPING_Y -5.0)"/>
+  <xacro:property name="quadratic_damping_z" value="$(optenv HERON_QUADRATIC_DAMPING_Z -15.0)"/>
+  <xacro:property name="quadratic_damping_roll" value="$(optenv HERON_QUADRATIC_DAMPING_ROLL -8.0)"/>
+  <xacro:property name="quadratic_damping_pitch" value="$(optenv HERON_QUADRATIC_DAMPING_PITCH -8.0)"/>
+  <xacro:property name="quadratic_damping_yaw" value="$(optenv HERON_QUADRATIC_DAMPING_YAW -8.0)"/>
   <xacro:macro name="heron_hydro_model" params="namespace">
     <!-- List of hydrodynamic models this robot's links -->
@@ -32,17 +50,17 @@
           <type>fossen</type>
           <added_mass>
-             0   0   0   0   0   0
-             0   0   0   0   0   0
-             0   0   0   0   0   0
-             0   0   0   0   0   0
-             0   0   0   0   0   0
-             0   0   0   0   0   0
+             ${added_mass_x}   0   0   0   0   0
+             0   ${added_mass_y}   0   0   0   0
+             0   0   ${added_mass_z}   0   0   0
+             0   0   0   ${added_mass_roll}   0   0
+             0   0   0   0   ${added_mass_pitch}   0
+             0   0   0   0   0   ${added_mass_yaw}
           </added_mass>
           <offset_added_mass>0</offset_added_mass>
           <linear_damping>
-                -25 -24 -150 -20 -20 -10
+                ${linear_damping_x} ${linear_damping_y} ${linear_damping_z} ${linear_damping_roll} ${linear_damping_pitch} ${linear_damping_yaw}
             </linear_damping>
             <quadratic_damping>
-              -5 -5 -15 -8 -8 -8
+              ${quadratic_damping_x} ${quadratic_damping_y} ${quadratic_damping_z} ${quadratic_damping_roll} ${quadratic_damping_pitch} ${quadratic_damping_yaw}
             </quadratic_damping>
             <!-- Sanity check -->

File: heron_description/urdf/heron.urdf.xacro (robot description, xacro)
@@ -29,4 +29,5 @@
   <xacro:arg name="namespace" default=""/>
   <xacro:arg name="suffix_ns" default="$(arg namespace)"/>
+  <xacro:property name="heron_fluid_density" value="$(optenv HERON_FLUID_DENSITY 997.7735)"/>
   <!-- Include the ROV macro file -->
   <xacro:include filename="$(find heron_description)/urdf/base.xacro"/>
@@ -38,5 +39,5 @@
     <gazebo>
       <plugin name="uuv_plugin" filename="libuuv_underwater_object_ros_plugin.so">
-        <fluid_density>997.7735</fluid_density>
+        <fluid_density>${heron_fluid_density}</fluid_density>
         <debug>$(arg debug)</debug>
         <xacro:heron_hydro_model namespace="$(arg suffix_ns)"/>

Commit message: Rename base inertial URDF link

File: heron_description/urdf/base.xacro (robot description, xacro)
@@ -71,6 +71,6 @@
       </collision>
     </link>
-    <!-- Dummy Link to contain the inertial information for base_link -->
-    <link name="${namespace}dummy_link">
+    <!-- Inertial link for base_link. -->
+    <link name="${namespace}base_inertia_link">
       <inertial>
         <mass value="${base_mass}" />
@@ -82,7 +82,7 @@
       </inertial>
     </link>
-    <joint name="dummy_to_base" type="fixed">
+    <joint name="base_inertia_joint" type="fixed">
       <parent link="${namespace}base_link" />
-      <child link="${namespace}dummy_link" />
+      <child link="${namespace}base_inertia_link" />
     </joint>
     <gazebo reference="${namespace}base_link">
