Commit message: Expose passive simulation disturbance parameters

File: heron_description/urdf/heron.urdf.xacro (robot description, xacro)
@@ -30,4 +30,17 @@
   <xacro:arg name="suffix_ns" default="$(arg namespace)"/>
   <xacro:property name="heron_fluid_density" value="$(optenv HERON_FLUID_DENSITY 997.7735)"/>
+  <xacro:property name="disturbance_force_mean_x" value="$(optenv HERON_DISTURBANCE_FORCE_MEAN_X 0.0)"/>
+  <xacro:property name="disturbance_force_mean_y" value="$(optenv HERON_DISTURBANCE_FORCE_MEAN_Y 0.0)"/>
+  <xacro:property name="disturbance_force_mean_z" value="$(optenv HERON_DISTURBANCE_FORCE_MEAN_Z 0.0)"/>
+  <xacro:property name="disturbance_force_amplitude_x" value="$(optenv HERON_DISTURBANCE_FORCE_AMPLITUDE_X 0.0)"/>
+  <xacro:property name="disturbance_force_amplitude_y" value="$(optenv HERON_DISTURBANCE_FORCE_AMPLITUDE_Y 0.0)"/>
+  <xacro:property name="disturbance_force_amplitude_z" value="$(optenv HERON_DISTURBANCE_FORCE_AMPLITUDE_Z 0.0)"/>
+  <xacro:property name="disturbance_torque_mean_x" value="$(optenv HERON_DISTURBANCE_TORQUE_MEAN_X 0.0)"/>
+  <xacro:property name="disturbance_torque_mean_y" value="$(optenv HERON_DISTURBANCE_TORQUE_MEAN_Y 0.0)"/>
+  <xacro:property name="disturbance_torque_mean_z" value="$(optenv HERON_DISTURBANCE_TORQUE_MEAN_Z 0.0)"/>
+  <xacro:property name="disturbance_torque_amplitude_x" value="$(optenv HERON_DISTURBANCE_TORQUE_AMPLITUDE_X 0.0)"/>
+  <xacro:property name="disturbance_torque_amplitude_y" value="$(optenv HERON_DISTURBANCE_TORQUE_AMPLITUDE_Y 0.0)"/>
+  <xacro:property name="disturbance_torque_amplitude_z" value="$(optenv HERON_DISTURBANCE_TORQUE_AMPLITUDE_Z 0.0)"/>
+  <xacro:property name="disturbance_period_sec" value="$(optenv HERON_DISTURBANCE_PERIOD_SEC 12.0)"/>
   <!-- Include the ROV macro file -->
   <xacro:include filename="$(find heron_description)/urdf/base.xacro"/>
@@ -59,4 +72,14 @@
     </plugin>
   </gazebo>
+  <gazebo>
+    <plugin name="passive_disturbance" filename="libPassiveDisturbancePlugin.so">
+      <bodyName>$(arg suffix_ns)base_link</bodyName>
+      <forceMean>${disturbance_force_mean_x} ${disturbance_force_mean_y} ${disturbance_force_mean_z}</forceMean>
+      <forceAmplitude>${disturbance_force_amplitude_x} ${disturbance_force_amplitude_y} ${disturbance_force_amplitude_z}</forceAmplitude>
+      <torqueMean>${disturbance_torque_mean_x} ${disturbance_torque_mean_y} ${disturbance_torque_mean_z}</torqueMean>
+      <torqueAmplitude>${disturbance_torque_amplitude_x} ${disturbance_torque_amplitude_y} ${disturbance_torque_amplitude_z}</torqueAmplitude>
+      <periodSec>${disturbance_period_sec}</periodSec>
+    </plugin>
+  </gazebo>
   <!-- Joint state publisher plugin -->
   <gazebo>

Commit message: fix: replace obsolete Heron hydrodynamics dependency

File: heron_description/urdf/heron.urdf.xacro (robot description, xacro)
@@ -29,5 +29,4 @@
   <xacro:arg name="namespace" default=""/>
   <xacro:arg name="suffix_ns" default="$(arg namespace)"/>
-  <xacro:property name="heron_fluid_density" value="$(optenv HERON_FLUID_DENSITY 997.7735)"/>
   <xacro:property name="disturbance_force_mean_x" value="$(optenv HERON_DISTURBANCE_FORCE_MEAN_X 0.0)"/>
   <xacro:property name="disturbance_force_mean_y" value="$(optenv HERON_DISTURBANCE_FORCE_MEAN_Y 0.0)"/>
@@ -43,16 +42,34 @@
   <xacro:property name="disturbance_torque_amplitude_z" value="$(optenv HERON_DISTURBANCE_TORQUE_AMPLITUDE_Z 0.0)"/>
   <xacro:property name="disturbance_period_sec" value="$(optenv HERON_DISTURBANCE_PERIOD_SEC 12.0)"/>
+  <xacro:property name="linear_damping_x" value="$(optenv HERON_LINEAR_DAMPING_X -25.0)"/>
+  <xacro:property name="linear_damping_y" value="$(optenv HERON_LINEAR_DAMPING_Y -24.0)"/>
+  <xacro:property name="linear_damping_z" value="$(optenv HERON_LINEAR_DAMPING_Z -150.0)"/>
+  <xacro:property name="linear_damping_roll" value="$(optenv HERON_LINEAR_DAMPING_ROLL -20.0)"/>
+  <xacro:property name="linear_damping_pitch" value="$(optenv HERON_LINEAR_DAMPING_PITCH -20.0)"/>
+  <xacro:property name="linear_damping_yaw" value="$(optenv HERON_LINEAR_DAMPING_YAW -10.0)"/>
+  <xacro:property name="quadratic_damping_x" value="$(optenv HERON_QUADRATIC_DAMPING_X -5.0)"/>
+  <xacro:property name="quadratic_damping_y" value="$(optenv HERON_QUADRATIC_DAMPING_Y -5.0)"/>
+  <xacro:property name="quadratic_damping_z" value="$(optenv HERON_QUADRATIC_DAMPING_Z -15.0)"/>
+  <xacro:property name="quadratic_damping_roll" value="$(optenv HERON_QUADRATIC_DAMPING_ROLL -8.0)"/>
+  <xacro:property name="quadratic_damping_pitch" value="$(optenv HERON_QUADRATIC_DAMPING_PITCH -8.0)"/>
+  <xacro:property name="quadratic_damping_yaw" value="$(optenv HERON_QUADRATIC_DAMPING_YAW -8.0)"/>
   <!-- Include the ROV macro file -->
   <xacro:include filename="$(find heron_description)/urdf/base.xacro"/>
-  <xacro:include filename="$(find heron_description)/urdf/gazebo.xacro"/>
   <!-- Create the heron -->
   <xacro:heron_base namespace="$(arg suffix_ns)">
-    <!-- The underwater object plugin is given as an input block parameter to
-     allow the addition of external models of manipulator units -->
+    <!-- Keep the surface vessel at its waterline with an owned Noetic/Gazebo
+         model. This replaces the obsolete external UUV Simulator plugin. -->
     <gazebo>
-      <plugin name="uuv_plugin" filename="libuuv_underwater_object_ros_plugin.so">
-        <fluid_density>${heron_fluid_density}</fluid_density>
-        <debug>$(arg debug)</debug>
-        <xacro:heron_hydro_model namespace="$(arg suffix_ns)"/>
+      <plugin name="surface_hydrodynamics" filename="libSurfaceHydrodynamicsPlugin.so">
+        <bodyName>$(arg suffix_ns)base_footprint</bodyName>
+        <equilibriumZ>0.0</equilibriumZ>
+        <heaveStiffness>900.0</heaveStiffness>
+        <heaveDamping>180.0</heaveDamping>
+        <rollStiffness>35.0</rollStiffness>
+        <pitchStiffness>35.0</pitchStiffness>
+        <linearDamping>${-linear_damping_x} ${-linear_damping_y} ${-linear_damping_z}</linearDamping>
+        <quadraticDamping>${-quadratic_damping_x} ${-quadratic_damping_y} ${-quadratic_damping_z}</quadraticDamping>
+        <angularDamping>${-linear_damping_roll} ${-linear_damping_pitch} ${-linear_damping_yaw}</angularDamping>
+        <angularQuadraticDamping>${-quadratic_damping_roll} ${-quadratic_damping_pitch} ${-quadratic_damping_yaw}</angularQuadraticDamping>
       </plugin>
     </gazebo>
